Commit message: Add collision to URDF

File: urdf/hokuyo_ust10lx.urdf.xacro (robot description, xacro)
@@ -12,4 +12,11 @@
         <material name="dark_grey" />
       </visual>
+      <collision>
+        <origin xyz="0 0 0" rpy="0 0 0" />
+        <geometry>
+          <!-- Origin of this mesh is the base of the bracket. -->
+          <mesh filename="package://generic_robot/meshes/hokuyo_ust10lx.stl" />
+        </geometry>
+      </collision>
       <inertial>
         <mass value="1.1" />

Commit message: Fix typo for package name

File: urdf/hokuyo_ust10lx.urdf.xacro (robot description, xacro)
@@ -16,5 +16,5 @@
         <geometry>
           <!-- Origin of this mesh is the base of the bracket. -->
-          <mesh filename="package://generic_robot/meshes/hokuyo_ust10lx.stl" />
+          <mesh filename="package://urg_node/meshes/hokuyo_ust10lx.stl" />
         </geometry>
       </collision>
