Commit message: Fix typo in package name

File: urdf/hokuyo_ust10.urdf.xacro (robot description, xacro)
@@ -58,5 +58,5 @@
         <geometry>
           <!-- Origin of this mesh is the base of the bracket. -->
-          <mesh filename="package://jackal_description/meshes/hokuyo_ust10.stl" />
+          <mesh filename="package://urg_node/meshes/hokuyo_ust10.stl" />
         </geometry>
         <material name="dark_grey" />
